File: mosfet_driver_8chan.sch (KiCad schematic (older format))
At the start: 67 parts, among them Q1 TSM3404, Q2 TSM3404, Q3 TSM3404, Q4 TSM3404, Q5 TSM3404, Q6 TSM3404, Q7 TSM3404, Q8 TSM3404, U1 EL817S1(B)(TU)-F, U2 EL817S1(B)(TU)-F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

Commit message: halfway routed
Parts:
- U1, U2, U3, U4, U5, U6, U7, U8: footprint Opto-Devices:Optocoupler_SMD_HandSoldering_KPC357_LTV35x_PC357_SingleChannel -> Octanis5-Rack_kicadlib:EL817S1-B-TU-F
Changed lines of the file:
@@
 F 0 "U1" H 1650 1975 50  0000 C CNN
 F 1 "EL817S1(B)(TU)-F" H 1650 1884 50  0000 C CNN
-F 2 "Opto-Devices:Optocoupler_SMD_HandSoldering_KPC357_LTV35x_PC357_SingleChannel" H 1650 1650 50  0001 C CNN
+F 2 "Octanis5-Rack_kicadlib:EL817S1-B-TU-F" H 1650 1650 50  0001 C CNN
 F 3 "" H 1650 1650 50  0001 C CNN
 F 4 "C63268" H 1650 1650 60  0001 C CNN "LCSC P/N"
@@
 F 0 "U2" H 1650 3875 50  0000 C CNN
 F 1 "EL817S1(B)(TU)-F" H 1650 3784 50  0000 C CNN
-F 2 "Opto-Devices:Optocoupler_SMD_HandSoldering_KPC357_LTV35x_PC357_SingleChannel" H 1650 3550 50  0001 C CNN
+F 2 "Octanis5-Rack_kicadlib:EL817S1-B-TU-F" H 1650 3550 50  0001 C CNN
 F 3 "" H 1650 3550 50  0001 C CNN
 F 4 "C63268" H 0   0   60  0001 C CNN "LCSC P/N"
@@
 F 0 "U3" H 1650 5725 50  0000 C CNN
 F 1 "EL817S1(B)(TU)-F" H 1650 5634 50  0000 C CNN
-F 2 "Opto-Devices:Optocoupler_SMD_HandSoldering_KPC357_LTV35x_PC357_SingleChannel" H 1650 5400 50  0001 C CNN
+F 2 "Octanis5-Rack_kicadlib:EL817S1-B-TU-F" H 1650 5400 50  0001 C CNN
 F 3 "" H 1650 5400 50  0001 C CNN
 F 4 "C63268" H 0   0   60  0001 C CNN "LCSC P/N"
@@
 F 0 "U4" H 5250 1975 50  0000 C CNN
 F 1 "EL817S1(B)(TU)-F" H 5250 1884 50  0000 C CNN
-F 2 "Opto-Devices:Optocoupler_SMD_HandSoldering_KPC357_LTV35x_PC357_SingleChannel" H 5250 1650 50  0001 C CNN
+F 2 "Octanis5-Rack_kicadlib:EL817S1-B-TU-F" H 5250 1650 50  0001 C CNN
 F 3 "" H 5250 1650 50  0001 C CNN
 F 4 "C63268" H 0   0   60  0001 C CNN "LCSC P/N"
@@
 F 0 "U5" H 5250 3875 50  0000 C CNN
 F 1 "EL817S1(B)(TU)-F" H 5250 3784 50  0000 C CNN
-F 2 "Opto-Devices:Optocoupler_SMD_HandSoldering_KPC357_LTV35x_PC357_SingleChannel" H 5250 3550 50  0001 C CNN
+F 2 "Octanis5-Rack_kicadlib:EL817S1-B-TU-F" H 5250 3550 50  0001 C CNN
 F 3 "" H 5250 3550 50  0001 C CNN
 F 4 "C63268" H 0   0   60  0001 C CNN "LCSC P/N"
@@
 F 0 "U6" H 5250 5725 50  0000 C CNN
 F 1 "EL817S1(B)(TU)-F" H 5250 5634 50  0000 C CNN
-F 2 "Opto-Devices:Optocoupler_SMD_HandSoldering_KPC357_LTV35x_PC357_SingleChannel" H 5250 5400 50  0001 C CNN
+F 2 "Octanis5-Rack_kicadlib:EL817S1-B-TU-F" H 5250 5400 50  0001 C CNN
 F 3 "" H 5250 5400 50  0001 C CNN
 F 4 "C63268" H 0   0   60  0001 C CNN "LCSC P/N"
@@
 F 0 "U7" H 8750 1975 50  0000 C CNN
 F 1 "EL817S1(B)(TU)-F" H 8750 1884 50  0000 C CNN
-F 2 "Opto-Devices:Optocoupler_SMD_HandSoldering_KPC357_LTV35x_PC357_SingleChannel" H 8750 1650 50  0001 C CNN
+F 2 "Octanis5-Rack_kicadlib:EL817S1-B-TU-F" H 8750 1650 50  0001 C CNN
 F 3 "" H 8750 1650 50  0001 C CNN
 F 4 "C63268" H 0   0   60  0001 C CNN "LCSC P/N"
@@
 F 0 "U8" H 8750 3875 50  0000 C CNN
 F 1 "EL817S1(B)(TU)-F" H 8750 3784 50  0000 C CNN
-F 2 "Opto-Devices:Optocoupler_SMD_HandSoldering_KPC357_LTV35x_PC357_SingleChannel" H 8750 3550 50  0001 C CNN
+F 2 "Octanis5-Rack_kicadlib:EL817S1-B-TU-F" H 8750 3550 50  0001 C CNN
 F 3 "" H 8750 3550 50  0001 C CNN
 F 4 "C63268" H 0   0   60  0001 C CNN "LCSC P/N"
