File: RPi_GPIO.sch (KiCad schematic (older format))
At the start: 1 part, among them J300 RPi_GPIO

Commit message: halfway routed
Connections:
- net labels added: IN1, IN2, IN3, IN4, IN5, IN6, IN7, IN8
- wire segments 20 -> 28
Changed lines of the file:
@@
 	1    0    0    -1
 $EndComp
+Text GLabel 9350 4600 2    60   Input ~ 0
+IN8
+Wire Wire Line
+	9350 4600 9200 4600
+Text GLabel 7150 4500 0    60   Input ~ 0
+IN6
+Text GLabel 7150 4400 0    60   Input ~ 0
+IN4
+Text GLabel 7150 4300 0    60   Input ~ 0
+IN3
+Text GLabel 7150 4200 0    60   Input ~ 0
+IN1
+Text GLabel 9350 4500 2    60   Input ~ 0
+IN7
+Text GLabel 9350 4400 2    60   Input ~ 0
+IN5
+Text GLabel 9350 4200 2    60   Input ~ 0
+IN2
+Wire Wire Line
+	9350 4200 9200 4200
+Wire Wire Line
+	9350 4400 9200 4400
+Wire Wire Line
+	9350 4500 9200 4500
+Wire Wire Line
+	7300 4200 7150 4200
+Wire Wire Line
+	7150 4300 7300 4300
+Wire Wire Line
+	7300 4400 7150 4400
+Wire Wire Line
+	7150 4500 7300 4500
 $EndSCHEMATC

Commit message: finished component placement
Changed lines of the file:
@@
 $EndComp
 Text GLabel 9350 4600 2    60   Input ~ 0
-IN8
+IN1
 Wire Wire Line
 	9350 4600 9200 4600
 Text GLabel 7150 4500 0    60   Input ~ 0
+IN3
+Text GLabel 7150 4400 0    60   Input ~ 0
+IN5
+Text GLabel 7150 4300 0    60   Input ~ 0
 IN6
-Text GLabel 7150 4400 0    60   Input ~ 0
+Text GLabel 7150 4200 0    60   Input ~ 0
+IN8
+Text GLabel 9350 4500 2    60   Input ~ 0
+IN2
+Text GLabel 9350 4400 2    60   Input ~ 0
 IN4
-Text GLabel 7150 4300 0    60   Input ~ 0
-IN3
-Text GLabel 7150 4200 0    60   Input ~ 0
-IN1
-Text GLabel 9350 4500 2    60   Input ~ 0
+Text GLabel 9350 4200 2    60   Input ~ 0
 IN7
-Text GLabel 9350 4400 2    60   Input ~ 0
-IN5
-Text GLabel 9350 4200 2    60   Input ~ 0
-IN2
 Wire Wire Line
 	9350 4200 9200 4200

Commit message: finished routing
Connections:
- net labels added: SENSE1, SENSE2, SENSE3, SENSE4, SENSE5, SENSE6, SENSE7, SENSE8
- wire segments 28 -> 41
Changed lines of the file:
@@
 Thru-Hole Connector
 $Comp
-L +5V #PWR01
+L +5V #PWR14
 U 1 1 5A2414FA
 P 9350 2700
-F 0 "#PWR01" H 9350 2550 50  0001 C CNN
+F 0 "#PWR14" H 9350 2550 50  0001 C CNN
 F 1 "+5V" V 9365 2828 50  0000 L CNN
 F 2 "" H 9350 2700 50  0001 C CNN
@@
 $EndComp
 $Comp
-L +5V #PWR02
+L +5V #PWR15
 U 1 1 5A241512
 P 9350 2800
-F 0 "#PWR02" H 9350 2650 50  0001 C CNN
+F 0 "#PWR15" H 9350 2650 50  0001 C CNN
 F 1 "+5V" V 9365 2928 50  0000 L CNN
 F 2 "" H 9350 2800 50  0001 C CNN
@@
 	9350 2800 9200 2800
 $Comp
-L GND #PWR03
+L GND #PWR16
 U 1 1 5A2415A9
 P 9350 2900
-F 0 "#PWR03" H 9350 2650 50  0001 C CNN
+F 0 "#PWR16" H 9350 2650 50  0001 C CNN
 F 1 "GND" V 9355 2772 50  0000 R CNN
 F 2 "" H 9350 2900 50  0001 C CNN
@@
 	9200 2900 9350 2900
 $Comp
-L GND #PWR04
+L GND #PWR17
 U 1 1 5A2415DF
 P 9350 3300
-F 0 "#PWR04" H 9350 3050 50  0001 C CNN
+F 0 "#PWR17" H 9350 3050 50  0001 C CNN
 F 1 "GND" V 9355 3172 50  0000 R CNN
 F 2 "" H 9350 3300 50  0001 C CNN
@@
 	9200 3300 9350 3300
 $Comp
-L GND #PWR05
+L GND #PWR18
 U 1 1 5A2415E8
 P 9350 3600
-F 0 "#PWR05" H 9350 3350 50  0001 C CNN
+F 0 "#PWR18" H 9350 3350 50  0001 C CNN
 F 1 "GND" V 9355 3472 50  0000 R CNN
 F 2 "" H 9350 3600 50  0001 C CNN
@@
 	9200 3600 9350 3600
 $Comp
-L GND #PWR06
+L GND #PWR19
 U 1 1 5A2415F1
 P 9350 4100
-F 0 "#PWR06" H 9350 3850 50  0001 C CNN
+F 0 "#PWR19" H 9350 3850 50  0001 C CNN
 F 1 "GND" V 9355 3972 50  0000 R CNN
 F 2 "" H 9350 4100 50  0001 C CNN
@@
 	9200 4100 9350 4100
 $Comp
-L GND #PWR07
+L GND #PWR20
 U 1 1 5A2415FA
 P 9350 4300
-F 0 "#PWR07" H 9350 4050 50  0001 C CNN
+F 0 "#PWR20" H 9350 4050 50  0001 C CNN
 F 1 "GND" V 9355 4172 50  0000 R CNN
 F 2 "" H 9350 4300 50  0001 C CNN
@@
 	9200 4300 9350 4300
 $Comp
-L GND #PWR08
+L GND #PWR13
 U 1 1 5A241635
 P 7150 4600
-F 0 "#PWR08" H 7150 4350 50  0001 C CNN
+F 0 "#PWR13" H 7150 4350 50  0001 C CNN
 F 1 "GND" V 7155 4472 50  0000 R CNN
 F 2 "" H 7150 4600 50  0001 C CNN
@@
 	7300 4600 7150 4600
 $Comp
-L GND #PWR09
+L GND #PWR12
 U 1 1 5A24165B
 P 7150 3900
-F 0 "#PWR09" H 7150 3650 50  0001 C CNN
+F 0 "#PWR12" H 7150 3650 50  0001 C CNN
 F 1 "GND" V 7155 3772 50  0000 R CNN
 F 2 "" H 7150 3900 50  0001 C CNN
@@
 	7300 3900 7150 3900
 $Comp
-L GND #PWR010
+L GND #PWR11
 U 1 1 5A241664
 P 7150 3100
-F 0 "#PWR010" H 7150 2850 50  0001 C CNN
+F 0 "#PWR11" H 7150 2850 50  0001 C CNN
 F 1 "GND" V 7155 2972 50  0000 R CNN
 F 2 "" H 7150 3100 50  0001 C CNN
@@
 	7300 3100 7150 3100
 $Comp
-L +5V #PWR011
+L +5V #PWR4
 U 1 1 5A251279
 P 4600 2700
-F 0 "#PWR011" H 4600 2550 50  0001 C CNN
+F 0 "#PWR4" H 4600 2550 50  0001 C CNN
 F 1 "+5V" V 4615 2828 50  0000 L CNN
 F 2 "" H 4600 2700 50  0001 C CNN
@@
 $EndComp
 $Comp
-L +5V #PWR012
+L +5V #PWR5
 U 1 1 5A25127F
 P 4600 2800
-F 0 "#PWR012" H 4600 2650 50  0001 C CNN
+F 0 "#PWR5" H 4600 2650 50  0001 C CNN
 F 1 "+5V" V 4615 2928 50  0000 L CNN
 F 2 "" H 4600 2800 50  0001 C CNN
@@
 	4600 2800 4450 2800
 $Comp
-L GND #PWR013
+L GND #PWR6
 U 1 1 5A251287
 P 4600 2900
-F 0 "#PWR013" H 4600 2650 50  0001 C CNN
+F 0 "#PWR6" H 4600 2650 50  0001 C CNN
 F 1 "GND" V 4605 2772 50  0000 R CNN
 F 2 "" H 4600 2900 50  0001 C CNN
@@
 	4450 2900 4600 2900
 $Comp
-L GND #PWR014
+L GND #PWR7
 U 1 1 5A25128E
 P 4600 3300
-F 0 "#PWR014" H 4600 3050 50  0001 C CNN
+F 0 "#PWR7" H 4600 3050 50  0001 C CNN
 F 1 "GND" V 4605 3172 50  0000 R CNN
 F 2 "" H 4600 3300 50  0001 C CNN
@@
 	4450 3300 4600 3300
 $Comp
-L GND #PWR015
+L GND #PWR8
 U 1 1 5A251295
 P 4600 3600
-F 0 "#PWR015" H 4600 3350 50  0001 C CNN
+F 0 "#PWR8" H 4600 3350 50  0001 C CNN
 F 1 "GND" V 4605 3472 50  0000 R CNN
 F 2 "" H 4600 3600 50  0001 C CNN
@@
 	4450 3600 4600 3600
 $Comp
-L GND #PWR016
+L GND #PWR9
 U 1 1 5A25129C
 P 4600 4100
-F 0 "#PWR016" H 4600 3850 50  0001 C CNN
+F 0 "#PWR9" H 4600 3850 50  0001 C CNN
 F 1 "GND" V 4605 3972 50  0000 R CNN
 F 2 "" H 4600 4100 50  0001 C CNN
@@
 	4450 4100 4600 4100
 $Comp
-L GND #PWR017
+L GND #PWR10
 U 1 1 5A2512A3
 P 4600 4300
-F 0 "#PWR017" H 4600 4050 50  0001 C CNN
+F 0 "#PWR10" H 4600 4050 50  0001 C CNN
 F 1 "GND" V 4605 4172 50  0000 R CNN
 F 2 "" H 4600 4300 50  0001 C CNN
@@
 	4450 4300 4600 4300
 $Comp
-L GND #PWR018
+L GND #PWR3
 U 1 1 5A2512AA
 P 2400 4600
-F 0 "#PWR018" H 2400 4350 50  0001 C CNN
+F 0 "#PWR3" H 2400 4350 50  0001 C CNN
 F 1 "GND" V 2405 4472 50  0000 R CNN
 F 2 "" H 2400 4600 50  0001 C CNN
@@
 	2550 4600 2400 4600
 $Comp
-L GND #PWR019
+L GND #PWR2
 U 1 1 5A2512B1
 P 2400 3900
-F 0 "#PWR019" H 2400 3650 50  0001 C CNN
+F 0 "#PWR2" H 2400 3650 50  0001 C CNN
 F 1 "GND" V 2405 3772 50  0000 R CNN
 F 2 "" H 2400 3900 50  0001 C CNN
@@
 	2550 3900 2400 3900
 $Comp
-L GND #PWR020
+L GND #PWR1
 U 1 1 5A2512B8
 P 2400 3100
-F 0 "#PWR020" H 2400 2850 50  0001 C CNN
+F 0 "#PWR1" H 2400 2850 50  0001 C CNN
 F 1 "GND" V 2405 2972 50  0000 R CNN
 F 2 "" H 2400 3100 50  0001 C CNN
@@
 Wire Wire Line
 	7150 4500 7300 4500
+Text GLabel 7100 3600 0    60   Input ~ 0
+SENSE1
+Text GLabel 7100 3700 0    60   Input ~ 0
+SENSE2
+Text GLabel 9350 3700 2    60   Input ~ 0
+SENSE3
+Text GLabel 7100 3800 0    60   Input ~ 0
+SENSE4
+Text GLabel 9350 3800 2    60   Input ~ 0
+SENSE5
+Text GLabel 7100 4000 0    60   Input ~ 0
+SENSE7
+Text GLabel 9350 3900 2    60   Input ~ 0
+SENSE6
+Text GLabel 9350 4000 2    60   Input ~ 0
+SENSE8
+Wire Wire Line
+	9350 3500 9200 3500
+Wire Wire Line
+	7100 3200 7300 3200
+Wire Wire Line
+	7300 3300 7100 3300
+Wire Wire Line
+	7100 3400 7300 3400
+Wire Wire Line
+	7100 3600 7300 3600
+Wire Wire Line
+	7100 3700 7300 3700
+Wire Wire Line
+	7100 3800 7300 3800
+Wire Wire Line
+	9200 3400 9350 3400
+Wire Wire Line
+	9350 4000 9200 4000
+Wire Wire Line
+	9350 3900 9200 3900
+Wire Wire Line
+	9350 3800 9200 3800
+Wire Wire Line
+	7100 4000 7300 4000
+Wire Wire Line
+	9350 3700 9200 3700
 $EndSCHEMATC

Commit message: finished routing
Parts:
- added R25, R26, R27, R28, R37, R38, R39, R40: 150k, Resistors_SMD:R_0603, symbol R
- added R29, R30, R31, R32, R33, R34, R35, R36: 33k, Resistors_SMD:R_0603, symbol R
Connections:
- wire segments 41 -> 49

Commit message: final PCB as ordered
Parts:
- J300: LCSC P/N (none) -> C50982
Changed lines of the file:
@@
 F 2 "RPi_Hat:Pin_Header_Straight_2x20" H 7500 2700 60  0001 C CNN
 F 3 "" H 7500 2700 60  0000 C CNN
+F 4 "C50982" H 7500 2700 60  0001 C CNN "LCSC P/N"
 	1    7500 2700
 	1    0    0    -1
