File: RPi_Hat.kicad_pcb (KiCad board)
At the start: 2 copper layers, 120 x 75 mm, 82 parts, among them J1 Barrel_Jack, J10 Audio-Jack-3_2Switches, J2 Audio-Jack-3, J3 Audio-Jack-3_2Switches, J300 RPi_GPIO, J4 Audio-Jack-3_2Switches, J5 Audio-Jack-3_2Switches, J6 Audio-Jack-3_2Switches, J7 Audio-Jack-3_2Switches, J8 Audio-Jack-3_2Switches, J9 Audio-Jack-3_2Switches, Q1 TSM3404, Q2 TSM3404, Q3 TSM3404, Q4 TSM3404, Q5 TSM3404, Q6 TSM3404, Q7 TSM3404, Q8 TSM3404, U1 EL817S1(B)(TU)-F, U2 EL817S1(B)(TU)-F, U3 EL817S1(B)(TU)-F, U4 EL817S1(B)(TU)-F, U5 EL817S1(B)(TU)-F, U6 EL817S1(B)(TU)-F, U7 EL817S1(B)(TU)-F, U8 EL817S1(B)(TU)-F

Commit message: halfway routed
Parts:
- D3, D7, R1, R10, R11, R12, R13, R14, R15, R16, R2, R3, R4, R5, R6, R7, R8, R9: moved to B.Cu
- J10, J7, J8, J9: value Audio-Jack-3_2Switches -> Audio-Jack-3; footprint Octanis5-Rack_kicadlib:PJ307 -> Octanis5-Rack_kicadlib:PJ-313D; moved to B.Cu
- J3, J4, J5, J6: value Audio-Jack-3_2Switches -> Audio-Jack-3; footprint Octanis5-Rack_kicadlib:PJ307 -> Octanis5-Rack_kicadlib:PJ-313D
- U1, U2, U3, U4, U5, U6, U7, U8: footprint Opto-Devices:Optocoupler_SMD_HandSoldering_KPC357_LTV35x_PC357_SingleChannel -> Octanis5-Rack_kicadlib:EL817S1-B-TU-F; moved to B.Cu
- moved Q1 215.9 mm to (-56.2, 14.2)
- moved Q2 215.9 mm to (-44.8, 1.56)
- moved Q3 215.9 mm to (-36.5, -5.04)
- moved Q5 215.9 mm to (-43.7, -5.04)
- moved Q6 215.9 mm to (-63.4, 10.8)
- moved Q7 215.9 mm to (-63.4, 17.4)
- moved Q8 215.9 mm to (-56.2, 7.61)
- moved Q4 158.0 mm to (-10.0, 30.0)
- moved R9 155.0 mm to (27.5, 27.5), turned to 90 degrees
- moved R1 144.8 mm to (28.0, 12.5), turned to 90 degrees
- moved R10 142.5 mm to (32.5, 27.5), turned to 90 degrees
- moved R2 138.8 mm to (33.0, 12.5), turned to 90 degrees
- moved R3 136.5 mm to (38.0, 12.5), turned to 90 degrees
- moved R12 136.1 mm to (42.5, 27.5), turned to 90 degrees
- moved C2 135.0 mm to (-9.00, 52.5)
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Connections:
- J300 pad 31: Net-(J300-Pad31) -> IN1
- J300 pad 32: Net-(J300-Pad32) -> IN2
- J300 pad 33: Net-(J300-Pad33) -> IN3
- J300 pad 35: Net-(J300-Pad35) -> IN4
- J300 pad 36: Net-(J300-Pad36) -> IN5
- J300 pad 37: Net-(J300-Pad37) -> IN6
- J300 pad 38: Net-(J300-Pad38) -> IN7
- J300 pad 40: Net-(J300-Pad40) -> IN8

Commit message: finished component placement
Parts:
- added ?: , RPi_Hat:RPi_Hat_Mounting_Hole, F.Cu at (32.5, 56.2)
- added ?: , RPi_Hat:RPi_Hat_Mounting_Hole, F.Cu at (-9.50, 0.75)
- added ?: , RPi_Hat:RPi_Hat_Mounting_Hole, F.Cu at (-9.50, 56.2)
- added J11: Screw_Terminal_1x03, Connectors_JST:JST_PH_B3B-PH-K_03x2.00mm_Straight, F.Cu at (-26.0, 49.5)
- added J12: Screw_Terminal_1x03, Connectors_JST:JST_PH_B3B-PH-K_03x2.00mm_Straight, F.Cu at (-26.0, 41.5)
- added J13: Screw_Terminal_1x03, Connectors_JST:JST_PH_B3B-PH-K_03x2.00mm_Straight, F.Cu at (-26.0, 33.5)
- added J14: Screw_Terminal_1x03, Connectors_JST:JST_PH_B3B-PH-K_03x2.00mm_Straight, F.Cu at (-26.0, 25.5)
- added J15: Screw_Terminal_1x03, Connectors_JST:JST_PH_B3B-PH-K_03x2.00mm_Straight, F.Cu at (-26.0, 17.5)
- added J16: Screw_Terminal_1x03, Connectors_JST:JST_PH_B3B-PH-K_03x2.00mm_Straight, F.Cu at (-26.0, 9.50)
- added J17: Screw_Terminal_1x03, Connectors_JST:JST_PH_B3B-PH-K_03x2.00mm_Straight, F.Cu at (-26.0, 1.50)
- added J18: Screw_Terminal_1x03, Connectors_JST:JST_PH_B3B-PH-K_03x2.00mm_Straight, F.Cu at (-26.0, -6.50)
- D1, D10, D11, D12, D13, D14, D15, D16, D2, D25, D4, D5, D6, D8, D9, J1, Q1, Q2, Q3, Q4, Q5, Q6, Q7, Q8, R17, R18, R19, R20, R21, R22, R23, R24: moved to B.Cu
- J2: footprint Octanis5-Rack_kicadlib:PJ307 -> Octanis5-Rack_kicadlib:PJ-313D
- moved D16 196.3 mm to (-17.5, -2.50), turned to 180 degrees
- moved D24 178.5 mm to (8.00, 14.0), turned to 180 degrees
- moved R21 174.1 mm to (3.00, 29.0)
- moved D22 170.9 mm to (8.00, 24.0), turned to 180 degrees
- moved D18 169.5 mm to (8.00, 44.0), turned to 180 degrees
- moved D10 168.0 mm to (-7.50, 42.5), turned to 180 degrees
- moved D23 166.2 mm to (8.00, 19.0), turned to 180 degrees
- moved R18 163.2 mm to (3.00, 44.0)
- moved D20 163.2 mm to (8.00, 34.0), turned to 180 degrees
- moved D17 162.3 mm to (8.00, 49.0), turned to 180 degrees
- moved D11 161.8 mm to (-7.50, 35.0), turned to 180 degrees
- moved R23 161.5 mm to (3.00, 19.0)
- moved D21 157.8 mm to (8.00, 29.0), turned to 180 degrees
- moved D15 157.7 mm to (-17.5, 5.00), turned to 180 degrees
- moved D14 157.1 mm to (-7.50, 12.5), turned to 180 degrees
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Connections:
- J10 pad 3: GND -> VAA
- J3 pad 3: GND -> VAA
- J300 pad 31: IN1 -> IN8
- J300 pad 32: IN2 -> IN7
- J300 pad 33: IN3 -> IN6
- J300 pad 35: IN4 -> IN5
- J300 pad 36: IN5 -> IN4
- J300 pad 37: IN6 -> IN3
- J300 pad 38: IN7 -> IN2
- J300 pad 40: IN8 -> IN1
- J4 pad 3: GND -> VAA
- J5 pad 3: GND -> VAA
- J6 pad 3: GND -> VAA
- J7 pad 3: GND -> VAA
- J8 pad 3: GND -> VAA
- J9 pad 3: GND -> VAA
Other:
- outline, holes or cut-outs redrawn
- board text added: "<- mount PH connectors on this side!"

Commit message: finished routing
Parts:
- added C3: C, Capacitors_SMD:C_0805, B.Cu at (77.5, -4.50)
- added C4: C, Capacitors_SMD:C_0805, B.Cu at (12.5, -0.50)
Connections:
- J300 pad 19: Net-(J300-Pad19) -> SENSE1
- J300 pad 21: Net-(J300-Pad21) -> SENSE2
- J300 pad 22: Net-(J300-Pad22) -> SENSE3
- J300 pad 23: Net-(J300-Pad23) -> SENSE4
- J300 pad 24: Net-(J300-Pad24) -> SENSE5
- J300 pad 26: Net-(J300-Pad26) -> SENSE6
- J300 pad 27: Net-(J300-Pad27) -> SENSE7
- J300 pad 28: Net-(J300-Pad28) -> SENSE8
Routing:
- net VAA: track 0.00 -> 402.8 mm, vias 0 -> 18
- net GND: track 0.00 -> 146.3 mm, vias 0 -> 33
- net V_opto: track 0.00 -> 138.8 mm
- net SENSE5: track 0.00 -> 121.7 mm, vias 0 -> 2
- net SENSE7: track 0.00 -> 119.4 mm, vias 0 -> 3
- net SENSE6: track 0.00 -> 118.2 mm, vias 0 -> 2
- net SENSE1: track 0.00 -> 115.3 mm
- net SENSE2: track 0.00 -> 109.6 mm
- net SENSE3: track 0.00 -> 100.1 mm
- net SENSE4: track 0.00 -> 96.8 mm
- net SENSE8: track 0.00 -> 96.3 mm, vias 0 -> 2
- net +5V: track 0.00 -> 85.1 mm
- net OUT6: track 0.00 -> 84.7 mm, vias 0 -> 3
- net OUT5: track 0.00 -> 83.1 mm, vias 0 -> 3
- net OUT7: track 0.00 -> 75.6 mm, vias 0 -> 3
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- added copper zone on F.Cu, net GND
Other:
- net class Default: clearance 0.2 -> 0.25; via_drill 0.4 -> 0.3
- net class Power added: clearance 0.3, trace_width 0.4, via_dia 0.9, via_drill 0.6
- rule trace_clearance: 0.2 -> 0.25
- rule trace_min: 0.01 -> 0.15
- rule via_min_size: 0.4 -> 0.6

Commit message: finished routing
Parts:
- added G***: LOGO, Octanis3:octanis_open_incubator_logo, F.Cu at (55.0, 28.0)
- added R25: 150k, Resistors_SMD:R_0603, B.Cu at (28.0, -1.00)
- added R26: 150k, Resistors_SMD:R_0603, B.Cu at (30.0, -1.00)
- added R27: 150k, Resistors_SMD:R_0603, B.Cu at (34.0, -1.00)
- added R28: 150k, Resistors_SMD:R_0603, B.Cu at (40.0, -1.00)
- added R29: 33k, Resistors_SMD:R_0603, B.Cu at (42.0, 9.00)
- added R30: 33k, Resistors_SMD:R_0603, B.Cu at (36.0, 9.00)
- added R31: 33k, Resistors_SMD:R_0603, B.Cu at (32.0, 9.00)
- added R32: 33k, Resistors_SMD:R_0603, B.Cu at (30.0, 9.00)
- added R33: 33k, Resistors_SMD:R_0603, B.Cu at (34.0, 9.00)
- added R34: 33k, Resistors_SMD:R_0603, B.Cu at (38.0, 9.00)
- added R35: 33k, Resistors_SMD:R_0603, B.Cu at (40.0, 9.00)
- added R36: 33k, Resistors_SMD:R_0603, B.Cu at (44.0, 9.00)
- added R37: 150k, Resistors_SMD:R_0603, B.Cu at (32.0, -1.00)
- added R38: 150k, Resistors_SMD:R_0603, B.Cu at (36.0, -1.00)
- added R39: 150k, Resistors_SMD:R_0603, B.Cu at (38.0, -1.00)
- added R40: 150k, Resistors_SMD:R_0603, B.Cu at (42.0, -1.00)
- moved C3 1.50 mm to (77.5, -6.00)
Connections:
- J300 pad 19: SENSE1 -> Net-(J300-Pad19)
- J300 pad 21: SENSE2 -> Net-(J300-Pad21)
- J300 pad 22: SENSE3 -> Net-(J300-Pad22)
- J300 pad 23: SENSE4 -> Net-(J300-Pad23)
- J300 pad 24: SENSE5 -> Net-(J300-Pad24)
- J300 pad 26: SENSE6 -> Net-(J300-Pad26)
- J300 pad 27: SENSE7 -> Net-(J300-Pad27)
- J300 pad 28: SENSE8 -> Net-(J300-Pad28)
Routing:
- net GND: track 146.3 -> 160.5 mm, vias 33 -> 41
- net Net-(J300-Pad21): track 0.00 -> 10.9 mm
- net Net-(J300-Pad19): track 0.00 -> 10.5 mm
- net Net-(J300-Pad22): track 0.00 -> 10.2 mm
- net Net-(J300-Pad23): track 0.00 -> 10.1 mm
- net Net-(J300-Pad28): track 0.00 -> 9.83 mm
- net Net-(J300-Pad26): track 0.00 -> 9.44 mm
- net Net-(J300-Pad27): track 0.00 -> 9.33 mm
- net Net-(J300-Pad24): track 0.00 -> 9.33 mm
- net SENSE2: track 109.6 -> 102.0 mm, vias 0 -> 1
- net SENSE1: track 115.3 -> 108.8 mm, vias 0 -> 1
- net SENSE4: track 96.8 -> 90.6 mm, vias 0 -> 1
- net SENSE7: track 119.4 -> 114.6 mm, vias 3 -> 4
- net SENSE3: track 100.1 -> 96.3 mm, vias 0 -> 1
- net SENSE5: track 121.7 -> 119.5 mm, vias 2 -> 3
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Other:
- board text added: "Octanis 5 Rack MOSFET driver board v1.0. racks.octanis.org"

Commit message: final PCB as ordered
Changed lines of the file:
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@@
 (kicad_pcb (version 20170123) (host pcbnew "(2017-06-12 revision 19d5cc754)-master")
   (general
-    (links 0)
-    (no_connects 19)
+    (links 239)
+    (no_connects 18)
     (area -37.550001 -15.7 134.078571 69.4825)
     (thickness 1.6)
     (drawings 69)
-    (tracks 962)
+    (tracks 964)
     (zones 0)
     (modules 112)
@@
     (trace_clearance 0.25)
     (zone_clearance 0.508)
-    (zone_45_only no)
+    (zone_45_only yes)
     (trace_min 0.15)
     (segment_width 0.1)
@@
     (pad_to_mask_clearance 0)
     (aux_axis_origin 0 0)
-    (grid_origin 74 -5)
+    (grid_origin 89 32.25)
     (visible_elements 7FFFFFFF)
     (pcbplotparams
-      (layerselection 0x00030_80000001)
-      (usegerberextensions false)
+      (layerselection 0x010f0_ffffffff)
+      (usegerberextensions true)
       (excludeedgelayer true)
       (linewidth 0.100000)
@@
   (segment (start 13.5 -0.5) (end 13.5 2.68) (width 0.9) (layer B.Cu) (net 2))
   (segment (start 13.5 2.68) (end 13.45 2.73) (width 0.9) (layer B.Cu) (net 2))
+  (segment (start -23.2 22.06151) (end -23.2 23.05) (width 0.4) (layer B.Cu) (net 3))
+  (segment (start -23.2 23.05) (end -22.75 23.5) (width 0.4) (layer B.Cu) (net 3))
+  (segment (start -22.75 23.5) (end -9.35116 23.5) (width 0.4) (layer B.Cu) (net 3))
+  (segment (start -9.35116 23.5) (end -5.35116 27.5) (width 0.4) (layer B.Cu) (net 3))
+  (segment (start -22.75 30.911509) (end -22.588491 30.75) (width 0.4) (layer B.Cu) (net 3))
+  (segment (start -22.588491 30.75) (end -9.70022 30.75) (width 0.4) (layer B.Cu) (net 3))
+  (segment (start -9.70022 30.75) (end -5.45022 35) (width 0.4) (layer B.Cu) (net 3))
+  (segment (start -5.45022 35) (end -5.35116 35) (width 0.4) (layer B.Cu) (net 3))
   (segment (start -23.2 38.56151) (end -23.2 37.45) (width 0.4) (layer F.Cu) (net 3))
   (segment (start -23.2 37.45) (end -22.75 37) (width 0.4) (layer F.Cu) (net 3))
@@
   (segment (start -22.78849 37) (end -22.25 37) (width 0.4) (layer B.Cu) (net 3))
   (segment (start -23.338491 30.911509) (end -22.75 30.911509) (width 0.4) (layer B.Cu) (net 3))
-  (segment (start -22.75 30.911509) (end -9.538711 30.911509) (width 0.4) (layer B.Cu) (net 3))
   (segment (start -23.2 32.06151) (end -23.199999 30.911509) (width 0.4) (layer B.Cu) (net 3))
   (segment (start -23.199999 30.911509) (end -22.75 30.911509) (width 0.4) (layer B.Cu) (net 3))
@@
   (segment (start -15.35116 5) (end -13.70148 5) (width 0.4) (layer B.Cu) (net 3))
   (segment (start -13.70148 5) (end -11.70148 7) (width 0.4) (layer B.Cu) (net 3))
-  (segment (start -23.2 22.06151) (end -23.199999 23.211511) (width 0.4) (layer B.Cu) (net 3))
-  (segment (start -23.199999 23.211511) (end -9.639649 23.211511) (width 0.4) (layer B.Cu) (net 3))
-  (segment (start -9.639649 23.211511) (end -5.35116 27.5) (width 0.4) (layer B.Cu) (net 3))
   (segment (start -26 21.5) (end -23.76151 21.5) (width 0.4) (layer B.Cu) (net 3))
   (segment (start -23.76151 21.5) (end -23.2 22.06151) (width 0.4) (layer B.Cu) (net 3))
   (segment (start -26 29.5) (end -24.75 29.5) (width 0.4) (layer B.Cu) (net 3))
   (segment (start -24.75 29.5) (end -23.338491 30.911509) (width 0.4) (layer B.Cu) (net 3))
-  (segment (start -9.538711 30.911509) (end -5.45022 35) (width 0.4) (layer B.Cu) (net 3))
-  (segment (start -5.45022 35) (end -5.35116 35) (width 0.4) (layer B.Cu) (net 3))
   (segment (start -9.95022 47) (end -5.45022 42.5) (width 0.4) (layer B.Cu) (net 3))
   (segment (start -5.45022 42.5) (end -5.35116 42.5) (width 0.4) (layer B.Cu) (net 3))
@@
     (connect_pads (clearance 0.508))
     (min_thickness 0.254)
-    (keepout (tracks not_allowed) (vias not_allowed) (copperpour allowed))
+    (keepout (tracks not_allowed) (vias not_allowed) (copperpour not_allowed))
     (fill (arc_segments 16) (thermal_gap 0.508) (thermal_bridge_width 0.508))
     (polygon
       (pts
-        (xy 31 -10.5) (xy 31 -6.5) (xy 32.5 -6.5) (xy 32.5 -11) (xy 31 -11)
+        (xy 40.75 -7.75) (xy 40.75 -3.75) (xy 42.25 -3.75) (xy 42.25 -8.25) (xy 40.75 -8.25)
       )
     )
