File: rack_driver_connectors.sch (KiCad schematic (older format))
At the start: 10 parts, among them J1 Barrel_Jack, J10 Audio-Jack-3_2Switches, J2 Audio-Jack-3, J3 Audio-Jack-3_2Switches, J4 Audio-Jack-3_2Switches, J5 Audio-Jack-3_2Switches, J6 Audio-Jack-3_2Switches, J7 Audio-Jack-3_2Switches, J8 Audio-Jack-3_2Switches, J9 Audio-Jack-3_2Switches

Commit message: halfway routed
Parts:
- removed J10, J3, J4, J5, J6, J7, J8, J9: Audio-Jack-3_2Switches, Octanis5-Rack_kicadlib:PJ307, symbol Audio-Jack-3_2Switches
- added J10, J3, J4, J5, J6, J7, J8, J9: Audio-Jack-3, Octanis5-Rack_kicadlib:PJ-313D, symbol Audio-Jack-3
Connections:
- net GND: now also J10.3, J3.3, J4.3, J5.3, J6.3, J7.3, J8.3, J9.3
- net OUT1: now also J3.2
- net OUT2: now also J4.2
- net OUT3: now also J5.2
- net OUT4: now also J6.2
- net OUT5: now also J7.2
- net OUT6: now also J8.2
- net OUT7: now also J9.2
- net OUT8: now also J10.2
- net SENSE1: now also J3.1
- net SENSE2: now also J4.1
- net SENSE3: now also J5.1
- net SENSE4: now also J6.1
- net SENSE5: now also J7.1
- net SENSE6: now also J8.1
- net SENSE7: now also J9.1
- net SENSE8: now also J10.1
Changed lines of the file:
@@
 Text GLabel 1600 1200 0    60   Input ~ 0
 OUT1
-$Comp
-L Audio-Jack-3_2Switches J3
-U 1 1 5A22DA0E
-P 2100 1100
-F 0 "J3" H 1813 1077 50  0000 R CNN
-F 1 "Audio-Jack-3_2Switches" H 1813 1168 50  0000 R CNN
-F 2 "Octanis5-Rack_kicadlib:PJ307" H 2350 1200 50  0001 C CNN
-F 3 "" H 2350 1200 50  0001 C CNN
-F 4 "C16684" H 2100 1100 60  0001 C CNN "LCSC P/N"
-	1    2100 1100
-	-1   0    0    1
-$EndComp
 Wire Wire Line
 	1600 1200 1900 1200
 Wire Wire Line
-	2300 900  2300 800
+	2300 800  2300 1000
 Wire Wire Line
 	2300 800  1600 800
@@
 	1600 2050 1900 2050
 Wire Wire Line
-	2300 1750 2300 1650
-Wire Wire Line
 	2300 1650 1600 1650
 $Comp
@@
 	1600 2850 1900 2850
 Wire Wire Line
-	2300 2550 2300 2450
+	2300 2450 2300 2650
 Wire Wire Line
 	2300 2450 1600 2450
@@
 	1600 3700 1900 3700
 Wire Wire Line
-	2300 3400 2300 3300
+	2300 3300 2300 3500
 Wire Wire Line
 	2300 3300 1600 3300
@@
 	1600 4550 1900 4550
 Wire Wire Line
-	2300 4250 2300 4150
+	2300 4150 2300 4350
 Wire Wire Line
 	2300 4150 1600 4150
@@
 	1600 5400 1900 5400
 Wire Wire Line
-	2300 5100 2300 5000
+	2300 5000 2300 5200
 Wire Wire Line
 	2300 5000 1600 5000
@@
 	1600 6200 1900 6200
 Wire Wire Line
-	2300 5900 2300 5800
+	2300 5800 2300 6000
 Wire Wire Line
 	2300 5800 1600 5800
@@
 	1600 7050 1900 7050
 Wire Wire Line
-	2300 6750 2300 6650
+	2300 6650 2300 6850
 Wire Wire Line
 	2300 6650 1600 6650
@@
 Wire Wire Line
 	1600 6950 1900 6950
-$Comp
-L Audio-Jack-3_2Switches J4
-U 1 1 5A240485
-P 2100 1950
-F 0 "J4" H 1813 1927 50  0000 R CNN
-F 1 "Audio-Jack-3_2Switches" H 1813 2018 50  0000 R CNN
-F 2 "Octanis5-Rack_kicadlib:PJ307" H 2350 2050 50  0001 C CNN
-F 3 "" H 2350 2050 50  0001 C CNN
-F 4 "C16684" H 2100 1950 60  0001 C CNN "LCSC P/N"
-	1    2100 1950
-	-1   0    0    1
-$EndComp
-$Comp
-L Audio-Jack-3_2Switches J5
-U 1 1 5A2404AD
-P 2100 2750
-F 0 "J5" H 1813 2727 50  0000 R CNN
-F 1 "Audio-Jack-3_2Switches" H 1813 2818 50  0000 R CNN
-F 2 "Octanis5-Rack_kicadlib:PJ307" H 2350 2850 50  0001 C CNN
-F 3 "" H 2350 2850 50  0001 C CNN
-F 4 "C16684" H 2100 2750 60  0001 C CNN "LCSC P/N"
-	1    2100 2750
-	-1   0    0    1
-$EndComp
-$Comp
-L Audio-Jack-3_2Switches J6
-U 1 1 5A2404CD
-P 2100 3600
-F 0 "J6" H 1813 3577 50  0000 R CNN
-F 1 "Audio-Jack-3_2Switches" H 1813 3668 50  0000 R CNN
-F 2 "Octanis5-Rack_kicadlib:PJ307" H 2350 3700 50  0001 C CNN
-F 3 "" H 2350 3700 50  0001 C CNN
-F 4 "C16684" H 2100 3600 60  0001 C CNN "LCSC P/N"
-	1    2100 3600
-	-1   0    0    1
-$EndComp
-$Comp
-L Audio-Jack-3_2Switches J7
-U 1 1 5A2404F8
-P 2100 4450
-F 0 "J7" H 1813 4427 50  0000 R CNN
-F 1 "Audio-Jack-3_2Switches" H 1813 4518 50  0000 R CNN
-F 2 "Octanis5-Rack_kicadlib:PJ307" H 2350 4550 50  0001 C CNN
-F 3 "" H 2350 4550 50  0001 C CNN
-F 4 "C16684" H 2100 4450 60  0001 C CNN "LCSC P/N"
-	1    2100 4450
-	-1   0    0    1
-$EndComp
-$Comp
-L Audio-Jack-3_2Switches J8
-U 1 1 5A240556
-P 2100 5300
-F 0 "J8" H 1813 5277 50  0000 R CNN
-F 1 "Audio-Jack-3_2Switches" H 1813 5368 50  0000 R CNN
-F 2 "Octanis5-Rack_kicadlib:PJ307" H 2350 5400 50  0001 C CNN
-F 3 "" H 2350 5400 50  0001 C CNN
-F 4 "C16684" H 2100 5300 60  0001 C CNN "LCSC P/N"
-	1    2100 5300
-	-1   0    0    1
-$EndComp
-$Comp
-L Audio-Jack-3_2Switches J9
-U 1 1 5A240583
-P 2100 6100
-F 0 "J9" H 1813 6077 50  0000 R CNN
-F 1 "Audio-Jack-3_2Switches" H 1813 6168 50  0000 R CNN
-F 2 "Octanis5-Rack_kicadlib:PJ307" H 2350 6200 50  0001 C CNN
-F 3 "" H 2350 6200 50  0001 C CNN
-F 4 "C16684" H 2100 6100 60  0001 C CNN "LCSC P/N"
-	1    2100 6100
-	-1   0    0    1
-$EndComp
-$Comp
-L Audio-Jack-3_2Switches J10
-U 1 1 5A2405AE
-P 2100 6950
-F 0 "J10" H 1813 6927 50  0000 R CNN
-F 1 "Audio-Jack-3_2Switches" H 1813 7018 50  0000 R CNN
-F 2 "Octanis5-Rack_kicadlib:PJ307" H 2350 7050 50  0001 C CNN
-F 3 "" H 2350 7050 50  0001 C CNN
-F 4 "C16684" H 2100 6950 60  0001 C CNN "LCSC P/N"
-	1    2100 6950
-	-1   0    0    1
-$EndComp
 $Comp
 L GND #PWR064
@@
 Wire Wire Line
 	5900 1800 5900 1750
+$Comp
+L Audio-Jack-3 J3
+U 1 1 5A25B836
+P 2100 1100
+F 0 "J3" H 1813 1077 50  0000 R CNN
+F 1 "Audio-Jack-3" H 1813 1168 50  0000 R CNN
+F 2 "Octanis5-Rack_kicadlib:PJ-313D" H 2350 1200 50  0001 C CNN
+F 3 "" H 2350 1200 50  0001 C CNN
+F 4 "C95463" H 2100 1100 60  0001 C CNN "LCSC P/N"
+	1    2100 1100
+	-1   0    0    1
+$EndComp
+$Comp
+L Audio-Jack-3 J4
+U 1 1 5A25C2B1
+P 2100 1950
+F 0 "J4" H 1813 1927 50  0000 R CNN
+F 1 "Audio-Jack-3" H 1813 2018 50  0000 R CNN
+F 2 "Octanis5-Rack_kicadlib:PJ-313D" H 2350 2050 50  0001 C CNN
+F 3 "" H 2350 2050 50  0001 C CNN
+F 4 "C95463" H 2100 1950 60  0001 C CNN "LCSC P/N"
+	1    2100 1950
+	-1   0    0    1
+$EndComp
+Wire Wire Line
+	2300 1650 2300 1850
+$Comp
+L Audio-Jack-3 J5
+U 1 1 5A25C33B
+P 2100 2750
+F 0 "J5" H 1813 2727 50  0000 R CNN
+F 1 "Audio-Jack-3" H 1813 2818 50  0000 R CNN
+F 2 "Octanis5-Rack_kicadlib:PJ-313D" H 2350 2850 50  0001 C CNN
+F 3 "" H 2350 2850 50  0001 C CNN
+F 4 "C95463" H 2100 2750 60  0001 C CNN "LCSC P/N"
+	1    2100 2750
+	-1   0    0    1
+$EndComp
+$Comp
+L Audio-Jack-3 J6
+U 1 1 5A25C484
+P 2100 3600
+F 0 "J6" H 1813 3577 50  0000 R CNN
+F 1 "Audio-Jack-3" H 1813 3668 50  0000 R CNN
+F 2 "Octanis5-Rack_kicadlib:PJ-313D" H 2350 3700 50  0001 C CNN
+F 3 "" H 2350 3700 50  0001 C CNN
+F 4 "C95463" H 2100 3600 60  0001 C CNN "LCSC P/N"
+	1    2100 3600
+	-1   0    0    1
+$EndComp
+$Comp
+L Audio-Jack-3 J7
+U 1 1 5A25C65A
+P 2100 4450
+F 0 "J7" H 1813 4427 50  0000 R CNN
+F 1 "Audio-Jack-3" H 1813 4518 50  0000 R CNN
+F 2 "Octanis5-Rack_kicadlib:PJ-313D" H 2350 4550 50  0001 C CNN
+F 3 "" H 2350 4550 50  0001 C CNN
+F 4 "C95463" H 2100 4450 60  0001 C CNN "LCSC P/N"
+	1    2100 4450
+	-1   0    0    1
+$EndComp
+$Comp
+L Audio-Jack-3 J8
+U 1 1 5A25C736
+P 2100 5300
+F 0 "J8" H 1813 5277 50  0000 R CNN
+F 1 "Audio-Jack-3" H 1813 5368 50  0000 R CNN
+F 2 "Octanis5-Rack_kicadlib:PJ-313D" H 2350 5400 50  0001 C CNN
+F 3 "" H 2350 5400 50  0001 C CNN
+F 4 "C95463" H 2100 5300 60  0001 C CNN "LCSC P/N"
+	1    2100 5300
+	-1   0    0    1
+$EndComp
+$Comp
+L Audio-Jack-3 J9
+U 1 1 5A25C831
+P 2100 6100
+F 0 "J9" H 1813 6077 50  0000 R CNN
+F 1 "Audio-Jack-3" H 1813 6168 50  0000 R CNN
+F 2 "Octanis5-Rack_kicadlib:PJ-313D" H 2350 6200 50  0001 C CNN
+F 3 "" H 2350 6200 50  0001 C CNN
+F 4 "C95463" H 2100 6100 60  0001 C CNN "LCSC P/N"
+	1    2100 6100
+	-1   0    0    1
+$EndComp
+$Comp
+L Audio-Jack-3 J10
+U 1 1 5A25C8E8
+P 2100 6950
+F 0 "J10" H 1813 6927 50  0000 R CNN
+F 1 "Audio-Jack-3" H 1813 7018 50  0000 R CNN
+F 2 "Octanis5-Rack_kicadlib:PJ-313D" H 2350 7050 50  0001 C CNN
+F 3 "" H 2350 7050 50  0001 C CNN
+F 4 "C95463" H 2100 6950 60  0001 C CNN "LCSC P/N"
+	1    2100 6950
+	-1   0    0    1
+$EndComp
 $EndSCHEMATC

Commit message: finished component placement
Parts:
- added J11, J12, J13, J14, J15, J16, J17, J18: Screw_Terminal_1x03, Connectors_JST:JST_PH_B3B-PH-K_03x2.00mm_Straight, symbol Screw_Terminal_1x03
- J2: footprint Octanis5-Rack_kicadlib:PJ307 -> Octanis5-Rack_kicadlib:PJ-313D; LCSC P/N C16684 -> C95463
Connections:
- net GND: no longer J10.3, J3.3, J4.3, J5.3, J6.3, J7.3, J8.3, J9.3
- net OUT1: now also J11.1
- net OUT2: now also J12.1
- net OUT3: now also J13.1
- net OUT4: now also J14.1
- net OUT5: now also J15.1
- net OUT6: now also J16.1
- net OUT7: now also J17.1
- net OUT8: now also J18.1
- net SENSE1: now also J11.2
- net SENSE2: now also J12.2
- net SENSE3: now also J13.2
- net SENSE4: now also J14.2
- net SENSE5: now also J15.2
- net SENSE6: now also J16.2
- net SENSE7: now also J17.2
- net SENSE8: now also J18.2
- net VAA: now also J10.3, J3.3, J4.3, J5.3, J6.3, J7.3, J8.3, J9.3, J11.3, J12.3, J13.3, J14.3, J15.3, J16.3, J17.3, J18.3

Commit message: finished routing
Parts:
- added C3, C4: C, Capacitors_SMD:C_0805, symbol C
Connections:
- net +5V: now also C3.1, C4.1
- net GND: now also C3.2, C4.2
Changed lines of the file:
@@
 SENSE8
 $Comp
-L GND #PWR056
+L GND #PWR75
 U 1 1 5A240A33
 P 5400 1150
-F 0 "#PWR056" H 5400 900 50  0001 C CNN
+F 0 "#PWR75" H 5400 900 50  0001 C CNN
 F 1 "GND" V 5405 1022 50  0000 R CNN
 F 2 "" H 5400 1150 50  0001 C CNN
@@
 $EndComp
 $Comp
-L VAA #PWR057
+L VAA #PWR74
 U 1 1 5A240AA1
 P 5400 950
-F 0 "#PWR057" H 5400 800 50  0001 C CNN
+F 0 "#PWR74" H 5400 800 50  0001 C CNN
 F 1 "VAA" V 5418 1077 50  0000 L CNN
 F 2 "" H 5400 950 50  0001 C CNN
@@
 $EndComp
 $Comp
-L GND #PWR058
+L GND #PWR72
 U 1 1 5A2439C3
 P 5350 1750
-F 0 "#PWR058" H 5350 1500 50  0001 C CNN
+F 0 "#PWR72" H 5350 1500 50  0001 C CNN
 F 1 "GND" V 5355 1622 50  0000 R CNN
 F 2 "" H 5350 1750 50  0001 C CNN
@@
 $EndComp
 $Comp
-L +5V #PWR059
+L +5V #PWR73
 U 1 1 5A243A03
 P 5350 1900
-F 0 "#PWR059" H 5350 1750 50  0001 C CNN
+F 0 "#PWR73" H 5350 1750 50  0001 C CNN
 F 1 "+5V" V 5365 2028 50  0000 L CNN
 F 2 "" H 5350 1900 50  0001 C CNN
 F 3 "" H 5350 1900 50  0001 C CNN
 	1    5350 1900
-	0    -1   -1   0
+	0    -1   1    0
 $EndComp
 $Comp
@@
 $EndComp
 $Comp
-L VAA #PWR060
+L VAA #PWR56
 U 1 1 5A2B1208
 P 1600 800
-F 0 "#PWR060" H 1600 650 50  0001 C CNN
+F 0 "#PWR56" H 1600 650 50  0001 C CNN
 F 1 "VAA" V 1618 927 50  0000 L CNN
 F 2 "" H 1600 800 50  0001 C CNN
@@
 $EndComp
 $Comp
-L VAA #PWR061
+L VAA #PWR57
 U 1 1 5A2B1A55
 P 1600 1650
-F 0 "#PWR061" H 1600 1500 50  0001 C CNN
+F 0 "#PWR57" H 1600 1500 50  0001 C CNN
 F 1 "VAA" V 1618 1777 50  0000 L CNN
 F 2 "" H 1600 1650 50  0001 C CNN
@@
 $EndComp
 $Comp
-L VAA #PWR062
+L VAA #PWR58
 U 1 1 5A2B1A84
 P 1600 2450
-F 0 "#PWR062" H 1600 2300 50  0001 C CNN
+F 0 "#PWR58" H 1600 2300 50  0001 C CNN
 F 1 "VAA" V 1618 2577 50  0000 L CNN
 F 2 "" H 1600 2450 50  0001 C CNN
@@
 $EndComp
 $Comp
-L VAA #PWR063
+L VAA #PWR59
 U 1 1 5A2B1AB3
 P 1600 3300
-F 0 "#PWR063" H 1600 3150 50  0001 C CNN
+F 0 "#PWR59" H 1600 3150 50  0001 C CNN
 F 1 "VAA" V 1618 3427 50  0000 L CNN
 F 2 "" H 1600 3300 50  0001 C CNN
@@
 $EndComp
 $Comp
-L VAA #PWR064
+L VAA #PWR60
 U 1 1 5A2B1AE2
 P 1600 4150
-F 0 "#PWR064" H 1600 4000 50  0001 C CNN
+F 0 "#PWR60" H 1600 4000 50  0001 C CNN
 F 1 "VAA" V 1618 4277 50  0000 L CNN
 F 2 "" H 1600 4150 50  0001 C CNN
@@
 $EndComp
 $Comp
-L VAA #PWR065
+L VAA #PWR61
 U 1 1 5A2B1B11
 P 1600 5000
-F 0 "#PWR065" H 1600 4850 50  0001 C CNN
+F 0 "#PWR61" H 1600 4850 50  0001 C CNN
 F 1 "VAA" V 1618 5127 50  0000 L CNN
 F 2 "" H 1600 5000 50  0001 C CNN
@@
 $EndComp
 $Comp
-L VAA #PWR066
+L VAA #PWR62
 U 1 1 5A2B1B40
 P 1600 5800
-F 0 "#PWR066" H 1600 5650 50  0001 C CNN
+F 0 "#PWR62" H 1600 5650 50  0001 C CNN
 F 1 "VAA" V 1618 5927 50  0000 L CNN
 F 2 "" H 1600 5800 50  0001 C CNN
@@
 $EndComp
 $Comp
-L VAA #PWR067
+L VAA #PWR63
 U 1 1 5A2B1CA1
 P 1600 6650
-F 0 "#PWR067" H 1600 6500 50  0001 C CNN
+F 0 "#PWR63" H 1600 6500 50  0001 C CNN
 F 1 "VAA" V 1618 6777 50  0000 L CNN
 F 2 "" H 1600 6650 50  0001 C CNN
@@
 $EndComp
 $Comp
-L VAA #PWR068
+L VAA #PWR71
 U 1 1 5A2B1DA8
 P 3550 6650
-F 0 "#PWR068" H 3550 6500 50  0001 C CNN
+F 0 "#PWR71" H 3550 6500 50  0001 C CNN
 F 1 "VAA" V 3568 6777 50  0000 L CNN
 F 2 "" H 3550 6650 50  0001 C CNN
@@
 $EndComp
 $Comp
-L VAA #PWR069
+L VAA #PWR70
 U 1 1 5A2B1DD7
 P 3550 5800
-F 0 "#PWR069" H 3550 5650 50  0001 C CNN
+F 0 "#PWR70" H 3550 5650 50  0001 C CNN
 F 1 "VAA" V 3568 5927 50  0000 L CNN
 F 2 "" H 3550 5800 50  0001 C CNN
@@
 $EndComp
 $Comp
-L VAA #PWR070
+L VAA #PWR69
 U 1 1 5A2B1E06
 P 3550 5000
-F 0 "#PWR070" H 3550 4850 50  0001 C CNN
+F 0 "#PWR69" H 3550 4850 50  0001 C CNN
 F 1 "VAA" V 3568 5127 50  0000 L CNN
 F 2 "" H 3550 5000 50  0001 C CNN
@@
 $EndComp
 $Comp
-L VAA #PWR071
+L VAA #PWR68
 U 1 1 5A2B1E35
 P 3550 4150
-F 0 "#PWR071" H 3550 4000 50  0001 C CNN
+F 0 "#PWR68" H 3550 4000 50  0001 C CNN
 F 1 "VAA" V 3568 4277 50  0000 L CNN
 F 2 "" H 3550 4150 50  0001 C CNN
@@
 $EndComp
 $Comp
-L VAA #PWR072
+L VAA #PWR67
 U 1 1 5A2B1E64
 P 3550 3300
-F 0 "#PWR072" H 3550 3150 50  0001 C CNN
+F 0 "#PWR67" H 3550 3150 50  0001 C CNN
 F 1 "VAA" V 3568 3427 50  0000 L CNN
 F 2 "" H 3550 3300 50  0001 C CNN
@@
 $EndComp
 $Comp
-L VAA #PWR073
+L VAA #PWR66
 U 1 1 5A2B1E93
 P 3550 2450
-F 0 "#PWR073" H 3550 2300 50  0001 C CNN
+F 0 "#PWR66" H 3550 2300 50  0001 C CNN
 F 1 "VAA" V 3568 2577 50  0000 L CNN
 F 2 "" H 3550 2450 50  0001 C CNN
@@
 $EndComp
 $Comp
-L VAA #PWR074
+L VAA #PWR65
 U 1 1 5A2B214A
 P 3550 1650
-F 0 "#PWR074" H 3550 1500 50  0001 C CNN
+F 0 "#PWR65" H 3550 1500 50  0001 C CNN
 F 1 "VAA" V 3568 1777 50  0000 L CNN
 F 2 "" H 3550 1650 50  0001 C CNN
@@
 $EndComp
 $Comp
-L VAA #PWR075
+L VAA #PWR64
 U 1 1 5A2B2179
 P 3550 800
-F 0 "#PWR075" H 3550 650 50  0001 C CNN
+F 0 "#PWR64" H 3550 650 50  0001 C CNN
 F 1 "VAA" V 3568 927 50  0000 L CNN
 F 2 "" H 3550 800 50  0001 C CNN
@@
 	0    -1   -1   0
 $EndComp
+$Comp
+L C C3
+U 1 1 5A2B4C1D
+P 6800 1900
+F 0 "C3" H 6915 1946 50  0000 L CNN
+F 1 "C" H 6915 1855 50  0000 L CNN
+F 2 "Capacitors_SMD:C_0805" H 6838 1750 50  0001 C CNN
+F 3 "" H 6800 1900 50  0001 C CNN
+	1    6800 1900
+	1    0    0    -1
+$EndComp
+$Comp
+L C C4
+U 1 1 5A2B4D0C
+P 7200 1900
+F 0 "C4" H 7315 1946 50  0000 L CNN
+F 1 "C" H 7315 1855 50  0000 L CNN
+F 2 "Capacitors_SMD:C_0805" H 7238 1750 50  0001 C CNN
+F 3 "" H 7200 1900 50  0001 C CNN
+	1    7200 1900
+	1    0    0    -1
+$EndComp
+$Comp
+L +5V #PWR76
+U 1 1 5A2B4D61
+P 6800 1750
+F 0 "#PWR76" H 6800 1600 50  0001 C CNN
+F 1 "+5V" V 6815 1878 50  0000 L CNN
+F 2 "" H 6800 1750 50  0001 C CNN
+F 3 "" H 6800 1750 50  0001 C CNN
+	1    6800 1750
+	-1   0    0    -1
+$EndComp
+$Comp
+L +5V #PWR78
+U 1 1 5A2B4DA8
+P 7200 1750
+F 0 "#PWR78" H 7200 1600 50  0001 C CNN
+F 1 "+5V" V 7215 1878 50  0000 L CNN
+F 2 "" H 7200 1750 50  0001 C CNN
+F 3 "" H 7200 1750 50  0001 C CNN
+	1    7200 1750
+	-1   0    0    -1
+$EndComp
+$Comp
+L GND #PWR77
+U 1 1 5A2B4DDB
+P 6800 2050
+F 0 "#PWR77" H 6800 1800 50  0001 C CNN
+F 1 "GND" V 6805 1922 50  0000 R CNN
+F 2 "" H 6800 2050 50  0001 C CNN
+F 3 "" H 6800 2050 50  0001 C CNN
+	1    6800 2050
+	1    0    0    -1
+$EndComp
+$Comp
+L GND #PWR79
+U 1 1 5A2B4E4A
+P 7200 2050
+F 0 "#PWR79" H 7200 1800 50  0001 C CNN
+F 1 "GND" V 7205 1922 50  0000 R CNN
+F 2 "" H 7200 2050 50  0001 C CNN
+F 3 "" H 7200 2050 50  0001 C CNN
+	1    7200 2050
+	1    0    0    -1
+$EndComp
 $EndSCHEMATC

Commit message: finished routing
Parts:
- C3, C4: value C -> 10u
Changed lines of the file:
@@
 SENSE8
 $Comp
-L GND #PWR75
+L GND #PWR064
 U 1 1 5A240A33
 P 5400 1150
-F 0 "#PWR75" H 5400 900 50  0001 C CNN
+F 0 "#PWR064" H 5400 900 50  0001 C CNN
 F 1 "GND" V 5405 1022 50  0000 R CNN
 F 2 "" H 5400 1150 50  0001 C CNN
@@
 $EndComp
 $Comp
-L VAA #PWR74
+L VAA #PWR065
 U 1 1 5A240AA1
 P 5400 950
-F 0 "#PWR74" H 5400 800 50  0001 C CNN
+F 0 "#PWR065" H 5400 800 50  0001 C CNN
 F 1 "VAA" V 5418 1077 50  0000 L CNN
 F 2 "" H 5400 950 50  0001 C CNN
@@
 $EndComp
 $Comp
-L GND #PWR72
+L GND #PWR066
 U 1 1 5A2439C3
 P 5350 1750
-F 0 "#PWR72" H 5350 1500 50  0001 C CNN
+F 0 "#PWR066" H 5350 1500 50  0001 C CNN
 F 1 "GND" V 5355 1622 50  0000 R CNN
 F 2 "" H 5350 1750 50  0001 C CNN
@@
 $EndComp
 $Comp
-L +5V #PWR73
+L +5V #PWR067
 U 1 1 5A243A03
 P 5350 1900
-F 0 "#PWR73" H 5350 1750 50  0001 C CNN
+F 0 "#PWR067" H 5350 1750 50  0001 C CNN
 F 1 "+5V" V 5365 2028 50  0000 L CNN
 F 2 "" H 5350 1900 50  0001 C CNN
@@
 $EndComp
 $Comp
-L VAA #PWR56
+L VAA #PWR068
 U 1 1 5A2B1208
 P 1600 800
-F 0 "#PWR56" H 1600 650 50  0001 C CNN
+F 0 "#PWR068" H 1600 650 50  0001 C CNN
 F 1 "VAA" V 1618 927 50  0000 L CNN
 F 2 "" H 1600 800 50  0001 C CNN
@@
 $EndComp
 $Comp
-L VAA #PWR57
+L VAA #PWR069
 U 1 1 5A2B1A55
 P 1600 1650
-F 0 "#PWR57" H 1600 1500 50  0001 C CNN
+F 0 "#PWR069" H 1600 1500 50  0001 C CNN
 F 1 "VAA" V 1618 1777 50  0000 L CNN
 F 2 "" H 1600 1650 50  0001 C CNN
@@
 $EndComp
 $Comp
-L VAA #PWR58
+L VAA #PWR070
 U 1 1 5A2B1A84
 P 1600 2450
-F 0 "#PWR58" H 1600 2300 50  0001 C CNN
+F 0 "#PWR070" H 1600 2300 50  0001 C CNN
 F 1 "VAA" V 1618 2577 50  0000 L CNN
 F 2 "" H 1600 2450 50  0001 C CNN
@@
 $EndComp
 $Comp
-L VAA #PWR59
+L VAA #PWR071
 U 1 1 5A2B1AB3
 P 1600 3300
-F 0 "#PWR59" H 1600 3150 50  0001 C CNN
+F 0 "#PWR071" H 1600 3150 50  0001 C CNN
 F 1 "VAA" V 1618 3427 50  0000 L CNN
 F 2 "" H 1600 3300 50  0001 C CNN
@@
 $EndComp
 $Comp
-L VAA #PWR60
+L VAA #PWR072
 U 1 1 5A2B1AE2
 P 1600 4150
-F 0 "#PWR60" H 1600 4000 50  0001 C CNN
+F 0 "#PWR072" H 1600 4000 50  0001 C CNN
 F 1 "VAA" V 1618 4277 50  0000 L CNN
 F 2 "" H 1600 4150 50  0001 C CNN
@@
 $EndComp
 $Comp
-L VAA #PWR61
+L VAA #PWR073
 U 1 1 5A2B1B11
 P 1600 5000
-F 0 "#PWR61" H 1600 4850 50  0001 C CNN
+F 0 "#PWR073" H 1600 4850 50  0001 C CNN
 F 1 "VAA" V 1618 5127 50  0000 L CNN
 F 2 "" H 1600 5000 50  0001 C CNN
@@
 $EndComp
 $Comp
-L VAA #PWR62
+L VAA #PWR074
 U 1 1 5A2B1B40
 P 1600 5800
-F 0 "#PWR62" H 1600 5650 50  0001 C CNN
+F 0 "#PWR074" H 1600 5650 50  0001 C CNN
 F 1 "VAA" V 1618 5927 50  0000 L CNN
 F 2 "" H 1600 5800 50  0001 C CNN
@@
 $EndComp
 $Comp
-L VAA #PWR63
+L VAA #PWR075
 U 1 1 5A2B1CA1
 P 1600 6650
-F 0 "#PWR63" H 1600 6500 50  0001 C CNN
+F 0 "#PWR075" H 1600 6500 50  0001 C CNN
 F 1 "VAA" V 1618 6777 50  0000 L CNN
 F 2 "" H 1600 6650 50  0001 C CNN
@@
 $EndComp
 $Comp
-L VAA #PWR71
+L VAA #PWR076
 U 1 1 5A2B1DA8
 P 3550 6650
-F 0 "#PWR71" H 3550 6500 50  0001 C CNN
+F 0 "#PWR076" H 3550 6500 50  0001 C CNN
 F 1 "VAA" V 3568 6777 50  0000 L CNN
 F 2 "" H 3550 6650 50  0001 C CNN
@@
 $EndComp
 $Comp
-L VAA #PWR70
+L VAA #PWR077
 U 1 1 5A2B1DD7
 P 3550 5800
-F 0 "#PWR70" H 3550 5650 50  0001 C CNN
+F 0 "#PWR077" H 3550 5650 50  0001 C CNN
 F 1 "VAA" V 3568 5927 50  0000 L CNN
 F 2 "" H 3550 5800 50  0001 C CNN
@@
 $EndComp
 $Comp
-L VAA #PWR69
+L VAA #PWR078
 U 1 1 5A2B1E06
 P 3550 5000
-F 0 "#PWR69" H 3550 4850 50  0001 C CNN
+F 0 "#PWR078" H 3550 4850 50  0001 C CNN
 F 1 "VAA" V 3568 5127 50  0000 L CNN
 F 2 "" H 3550 5000 50  0001 C CNN
@@
 $EndComp
 $Comp
-L VAA #PWR68
+L VAA #PWR079
 U 1 1 5A2B1E35
 P 3550 4150
-F 0 "#PWR68" H 3550 4000 50  0001 C CNN
+F 0 "#PWR079" H 3550 4000 50  0001 C CNN
 F 1 "VAA" V 3568 4277 50  0000 L CNN
 F 2 "" H 3550 4150 50  0001 C CNN
@@
 $EndComp
 $Comp
-L VAA #PWR67
+L VAA #PWR080
 U 1 1 5A2B1E64
 P 3550 3300
-F 0 "#PWR67" H 3550 3150 50  0001 C CNN
+F 0 "#PWR080" H 3550 3150 50  0001 C CNN
 F 1 "VAA" V 3568 3427 50  0000 L CNN
 F 2 "" H 3550 3300 50  0001 C CNN
@@
 $EndComp
 $Comp
-L VAA #PWR66
+L VAA #PWR081
 U 1 1 5A2B1E93
 P 3550 2450
-F 0 "#PWR66" H 3550 2300 50  0001 C CNN
+F 0 "#PWR081" H 3550 2300 50  0001 C CNN
 F 1 "VAA" V 3568 2577 50  0000 L CNN
 F 2 "" H 3550 2450 50  0001 C CNN
@@
 $EndComp
 $Comp
-L VAA #PWR65
+L VAA #PWR082
 U 1 1 5A2B214A
 P 3550 1650
-F 0 "#PWR65" H 3550 1500 50  0001 C CNN
+F 0 "#PWR082" H 3550 1500 50  0001 C CNN
 F 1 "VAA" V 3568 1777 50  0000 L CNN
 F 2 "" H 3550 1650 50  0001 C CNN
@@
 $EndComp
 $Comp
-L VAA #PWR64
+L VAA #PWR083
 U 1 1 5A2B2179
 P 3550 800
-F 0 "#PWR64" H 3550 650 50  0001 C CNN
+F 0 "#PWR083" H 3550 650 50  0001 C CNN
 F 1 "VAA" V 3568 927 50  0000 L CNN
 F 2 "" H 3550 800 50  0001 C CNN
@@
 P 6800 1900
 F 0 "C3" H 6915 1946 50  0000 L CNN
-F 1 "C" H 6915 1855 50  0000 L CNN
+F 1 "10u" H 6915 1855 50  0000 L CNN
 F 2 "Capacitors_SMD:C_0805" H 6838 1750 50  0001 C CNN
 F 3 "" H 6800 1900 50  0001 C CNN
@@
 P 7200 1900
 F 0 "C4" H 7315 1946 50  0000 L CNN
-F 1 "C" H 7315 1855 50  0000 L CNN
+F 1 "10u" H 7315 1855 50  0000 L CNN
 F 2 "Capacitors_SMD:C_0805" H 7238 1750 50  0001 C CNN
 F 3 "" H 7200 1900 50  0001 C CNN
@@
 $EndComp
 $Comp
-L +5V #PWR76
+L +5V #PWR084
 U 1 1 5A2B4D61
 P 6800 1750
-F 0 "#PWR76" H 6800 1600 50  0001 C CNN
+F 0 "#PWR084" H 6800 1600 50  0001 C CNN
 F 1 "+5V" V 6815 1878 50  0000 L CNN
 F 2 "" H 6800 1750 50  0001 C CNN
@@
 $EndComp
 $Comp
-L +5V #PWR78
+L +5V #PWR085
 U 1 1 5A2B4DA8
 P 7200 1750
-F 0 "#PWR78" H 7200 1600 50  0001 C CNN
+F 0 "#PWR085" H 7200 1600 50  0001 C CNN
 F 1 "+5V" V 7215 1878 50  0000 L CNN
 F 2 "" H 7200 1750 50  0001 C CNN
@@
 $EndComp
 $Comp
-L GND #PWR77
+L GND #PWR086
 U 1 1 5A2B4DDB
 P 6800 2050
-F 0 "#PWR77" H 6800 1800 50  0001 C CNN
+F 0 "#PWR086" H 6800 1800 50  0001 C CNN
 F 1 "GND" V 6805 1922 50  0000 R CNN
 F 2 "" H 6800 2050 50  0001 C CNN
@@
 $EndComp
 $Comp
-L GND #PWR79
+L GND #PWR087
 U 1 1 5A2B4E4A
 P 7200 2050
-F 0 "#PWR79" H 7200 1800 50  0001 C CNN
+F 0 "#PWR087" H 7200 1800 50  0001 C CNN
 F 1 "GND" V 7205 1922 50  0000 R CNN
 F 2 "" H 7200 2050 50  0001 C CNN

Commit message: final PCB as ordered
Parts:
- C3, C4: LCSC P/N (none) -> C123631
Changed lines of the file:
@@
 F 2 "Capacitors_SMD:C_0805" H 6838 1750 50  0001 C CNN
 F 3 "" H 6800 1900 50  0001 C CNN
+F 4 "C123631" H 6800 1900 60  0001 C CNN "LCSC P/N"
 	1    6800 1900
 	1    0    0    -1
@@
 F 2 "Capacitors_SMD:C_0805" H 7238 1750 50  0001 C CNN
 F 3 "" H 7200 1900 50  0001 C CNN
+F 4 "C123631" H 7200 1900 60  0001 C CNN "LCSC P/N"
 	1    7200 1900
 	1    0    0    -1
